File: Hardware/PMS_2024/PMS/PMS.kicad_pcb (KiCad board)
At the start: 2 copper layers, 224 x 109.7 mm, 109 parts, among them J1 RJ45_LED_Shielded, Q1 BSS138, Q2 BSS138, Q3 BSS138, Q4 SPD30P06PGBTMA1, Q5 SPD30P06PGBTMA1, Q6 BSS138, Q7 IPB180N10S4-02, U1 Teensy4.1_DEV-16771, U2 OKI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

Commit message: created gerbs
Routing:
- net GND: vias 0 -> 3
Changed lines of the file:
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@@
       (outputformat 1)
       (mirror false)
-      (drillshape 1)
+      (drillshape 0)
       (scaleselection 1)
-      (outputdirectory "")
+      (outputdirectory "../../../Documentation/Gerbs/")
     )
   )
@@
     (fp_line (start 1.6 0.8) (end -1.6 0.8)
       (stroke (width 0.1) (type solid)) (layer "F.Fab"))
-    (pad "1" smd roundrect (at -1.5625 0 90) (size 1.325 1.8) (layers "F.Cu" "F.Paste" "F.Mask") (roundrect_rratio 0.188679)
+    (pad "1" smd roundrect (at -1.5625 0 90) (size 1.325 1.8) (layers "F.Cu" "F.Paste" "F.Mask") (roundrect_rratio 0.1886792453)
       (net 6 "NS_24V") (pintype "passive"))
-    (pad "2" smd roundrect (at 1.5625 0 90) (size 1.325 1.8) (layers "F.Cu" "F.Paste" "F.Mask") (roundrect_rratio 0.188679)
+    (pad "2" smd roundrect (at 1.5625 0 90) (size 1.325 1.8) (layers "F.Cu" "F.Paste" "F.Mask") (roundrect_rratio 0.1886792453)
       (net 4 "GND") (pintype "passive"))
     (model "${KICAD6_3DMODEL_DIR}/Capacitor_SMD.3dshapes/C_1206_3216Metric.wrl"
@@
     (fp_line (start 1.6 0.8) (end -1.6 0.8)
       (stroke (width 0.1) (type solid)) (layer "F.Fab"))
-    (pad "1" smd roundrect (at -1.5625 0 90) (size 1.325 1.8) (layers "F.Cu" "F.Paste" "F.Mask") (roundrect_rratio 0.188679)
+    (pad "1" smd roundrect (at -1.5625 0 90) (size 1.325 1.8) (layers "F.Cu" "F.Paste" "F.Mask") (roundrect_rratio 0.1886792453)
       (net 3 "POE_24V") (pintype "passive"))
-    (pad "2" smd roundrect (at 1.5625 0 90) (size 1.325 1.8) (layers "F.Cu" "F.Paste" "F.Mask") (roundrect_rratio 0.188679)
+    (pad "2" smd roundrect (at 1.5625 0 90) (size 1.325 1.8) (layers "F.Cu" "F.Paste" "F.Mask") (roundrect_rratio 0.1886792453)
       (net 4 "GND") (pintype "passive"))
     (model "${KICAD6_3DMODEL_DIR}/Capacitor_SMD.3dshapes/C_1206_3216Metric.wrl"
@@
     (pad "3" smd roundrect (at -7.65 -1.27 270) (size 4.6 0.8) (layers "F.Cu" "F.Paste" "F.Mask") (roundrect_rratio 0.25)
       (net 7 "PV") (pinfunction "S") (pintype "passive"))
-    (pad "4" smd roundrect (at -0.925 -2.775 270) (size 4.55 5.25) (layers "F.Cu" "F.Paste") (roundrect_rratio 0.054945)
+    (pad "4" smd roundrect (at -0.925 -2.775 270) (size 4.55 5.25) (layers "F.Cu" "F.Paste") (roundrect_rratio 0.05494505495)
       (net 9 "Motor_PWR") (pinfunction "D") (pintype "passive"))
-    (pad "4" smd roundrect (at -0.925 2.775 270) (size 4.55 5.25) (layers "F.Cu" "F.Paste") (roundrect_rratio 0.054945)
+    (pad "4" smd roundrect (at -0.925 2.775 270) (size 4.55 5.25) (layers "F.Cu" "F.Paste") (roundrect_rratio 0.05494505495)
       (net 9 "Motor_PWR") (pinfunction "D") (pintype "passive"))
-    (pad "4" smd roundrect (at 1.5 0 270) (size 9.4 10.8) (layers "F.Cu" "F.Mask") (roundrect_rratio 0.026596)
+    (pad "4" smd roundrect (at 1.5 0 270) (size 9.4 10.8) (layers "F.Cu" "F.Mask") (roundrect_rratio 0.02659595745)
       (net 9 "Motor_PWR") (pinfunction "D") (pintype "passive"))
-    (pad "4" smd roundrect (at 3.925 -2.775 270) (size 4.55 5.25) (layers "F.Cu" "F.Paste") (roundrect_rratio 0.054945)
+    (pad "4" smd roundrect (at 3.925 -2.775 270) (size 4.55 5.25) (layers "F.Cu" "F.Paste") (roundrect_rratio 0.05494505495)
       (net 9 "Motor_PWR") (pinfunction "D") (pintype "passive"))
-    (pad "4" smd roundrect (at 3.925 2.775 270) (size 4.55 5.25) (layers "F.Cu" "F.Paste") (roundrect_rratio 0.054945)
+    (pad "4" smd roundrect (at 3.925 2.775 270) (size 4.55 5.25) (layers "F.Cu" "F.Paste") (roundrect_rratio 0.05494505495)
       (net 9 "Motor_PWR") (pinfunction "D") (pintype "passive"))
     (pad "5" smd roundrect (at -7.65 1.27 270) (size 4.6 0.8) (layers "F.Cu" "F.Paste" "F.Mask") (roundrect_rratio 0.25)
@@
     (fp_line (start 1.6 0.8) (end -1.6 0.8)
       (stroke (width 0.1) (type solid)) (layer "F.Fab"))
-    (pad "1" smd roundrect (at -1.5625 0) (size 1.325 1.8) (layers "F.Cu" "F.Paste" "F.Mask") (roundrect_rratio 0.188679)
+    (pad "1" smd roundrect (at -1.5625 0) (size 1.325 1.8) (layers "F.Cu" "F.Paste" "F.Mask") (roundrect_rratio 0.1886792453)
       (net 7 "PV") (pintype "passive"))
-    (pad "2" smd roundrect (at 1.5625 0) (size 1.325 1.8) (layers "F.Cu" "F.Paste" "F.Mask") (roundrect_rratio 0.188679)
+    (pad "2" smd roundrect (at 1.5625 0) (size 1.325 1.8) (layers "F.Cu" "F.Paste" "F.Mask") (roundrect_rratio 0.1886792453)
       (net 4 "GND") (pintype "passive"))
     (model "${KICAD6_3DMODEL_DIR}/Capacitor_SMD.3dshapes/C_1206_3216Metric.wrl"
@@
     (fp_line (start 4.11 2.7) (end 3.11 2.7)
       (stroke (width 0.1) (type solid)) (layer "F.Fab"))
-    (pad "1" smd roundrect (at -5.04 -2.28 90) (size 2.2 1.2) (layers "F.Cu" "F.Paste" "F.Mask") (roundrect_rratio 0.208333)
+    (pad "1" smd roundrect (at -5.04 -2.28 90) (size 2.2 1.2) (layers "F.Cu" "F.Paste" "F.Mask") (roundrect_rratio 0.2083333333)
       (net 40 "Net-(Q4-G)") (pinfunction "G") (pintype "passive"))
-    (pad "2" smd roundrect (at -0.415 -1.525 90) (size 3.05 2.75) (layers "F.Cu" "F.Paste") (roundrect_rratio 0.090909)
+    (pad "2" smd roundrect (at -0.415 -1.525 90) (size 3.05 2.75) (layers "F.Cu" "F.Paste") (roundrect_rratio 0.09090909091)
       (net 11 "LowCurrent_PWR") (pinfunction "D") (pintype "passive"))
-    (pad "2" smd roundrect (at -0.415 1.525 90) (size 3.05 2.75) (layers "F.Cu" "F.Paste") (roundrect_rratio 0.090909)
+    (pad "2" smd roundrect (at -0.415 1.525 90) (size 3.05 2.75) (layers "F.Cu" "F.Paste") (roundrect_rratio 0.09090909091)
       (net 11 "LowCurrent_PWR") (pinfunction "D") (pintype "passive"))
-    (pad "2" smd roundrect (at 1.26 0 90) (size 6.4 5.8) (layers "F.Cu" "F.Mask") (roundrect_rratio 0.043103)
+    (pad "2" smd roundrect (at 1.26 0 90) (size 6.4 5.8) (layers "F.Cu" "F.Mask") (roundrect_rratio 0.04310293103)
       (net 11 "LowCurrent_PWR") (pinfunction "D") (pintype "passive"))
-    (pad "2" smd roundrect (at 2.935 -1.525 90) (size 3.05 2.75) (layers "F.Cu" "F.Paste") (roundrect_rratio 0.090909)
+    (pad "2" smd roundrect (at 2.935 -1.525 90) (size 3.05 2.75) (layers "F.Cu" "F.Paste") (roundrect_rratio 0.09090909091)
       (net 11 "LowCurrent_PWR") (pinfunction "D") (pintype "passive"))
-    (pad "2" smd roundrect (at 2.935 1.525 90) (size 3.05 2.75) (layers "F.Cu" "F.Paste") (roundrect_rratio 0.090909)
+    (pad "2" smd roundrect (at 2.935 1.525 90) (size 3.05 2.75) (layers "F.Cu" "F.Paste") (roundrect_rratio 0.09090909091)
       (net 11 "LowCurrent_PWR") (pinfunction "D") (pintype "passive"))
-    (pad "3" smd roundrect (at -5.04 2.28 90) (size 2.2 1.2) (layers "F.Cu" "F.Paste" "F.Mask") (roundrect_rratio 0.208333)
+    (pad "3" smd roundrect (at -5.04 2.28 90) (size 2.2 1.2) (layers "F.Cu" "F.Paste" "F.Mask") (roundrect_rratio 0.2083333333)
       (net 7 "PV") (pinfunction "S") (pintype "passive"))
     (model "${KICAD6_3DMODEL_DIR}/Package_TO_SOT_SMD.3dshapes/TO-252-2.wrl"
@@
     (fp_line (start 4.11 2.7) (end 3.11 2.7)
       (stroke (width 0.1) (type solid)) (layer "F.Fab"))
-    (pad "1" smd roundrect (at -5.04 -2.28 180) (size 2.2 1.2) (layers "F.Cu" "F.Paste" "F.Mask") (roundrect_rratio 0.208333)
+    (pad "1" smd roundrect (at -5.04 -2.28 180) (size 2.2 1.2) (layers "F.Cu" "F.Paste" "F.Mask") (roundrect_rratio 0.2083333333)
       (net 41 "Net-(Q5-G)") (pinfunction "G") (pintype "passive"))
-    (pad "2" smd roundrect (at -0.415 -1.525 180) (size 3.05 2.75) (layers "F.Cu" "F.Paste") (roundrect_rratio 0.090909)
+    (pad "2" smd roundrect (at -0.415 -1.525 180) (size 3.05 2.75) (layers "F.Cu" "F.Paste") (roundrect_rratio 0.09090909091)
       (net 45 "Net-(Q5-D)") (pinfunction "D") (pintype "passive"))
-    (pad "2" smd roundrect (at -0.415 1.525 180) (size 3.05 2.75) (layers "F.Cu" "F.Paste") (roundrect_rratio 0.090909)
+    (pad "2" smd roundrect (at -0.415 1.525 180) (size 3.05 2.75) (layers "F.Cu" "F.Paste") (roundrect_rratio 0.09090909091)
       (net 45 "Net-(Q5-D)") (pinfunction "D") (pintype "passive"))
-    (pad "2" smd roundrect (at 1.26 0 180) (size 6.4 5.8) (layers "F.Cu" "F.Mask") (roundrect_rratio 0.043103)
+    (pad "2" smd roundrect (at 1.26 0 180) (size 6.4 5.8) (layers "F.Cu" "F.Mask") (roundrect_rratio 0.04310293103)
       (net 45 "Net-(Q5-D)") (pinfunction "D") (pintype "passive"))
-    (pad "2" smd roundrect (at 2.935 -1.525 180) (size 3.05 2.75) (layers "F.Cu" "F.Paste") (roundrect_rratio 0.090909)
+    (pad "2" smd roundrect (at 2.935 -1.525 180) (size 3.05 2.75) (layers "F.Cu" "F.Paste") (roundrect_rratio 0.09090909091)
       (net 45 "Net-(Q5-D)") (pinfunction "D") (pintype "passive"))
-    (pad "2" smd roundrect (at 2.935 1.525 180) (size 3.05 2.75) (layers "F.Cu" "F.Paste") (roundrect_rratio 0.090909)
+    (pad "2" smd roundrect (at 2.935 1.525 180) (size 3.05 2.75) (layers "F.Cu" "F.Paste") (roundrect_rratio 0.09090909091)
       (net 45 "Net-(Q5-D)") (pinfunction "D") (pintype "passive"))
-    (pad "3" smd roundrect (at -5.04 2.28 180) (size 2.2 1.2) (layers "F.Cu" "F.Paste" "F.Mask") (roundrect_rratio 0.208333)
+    (pad "3" smd roundrect (at -5.04 2.28 180) (size 2.2 1.2) (layers "F.Cu" "F.Paste" "F.Mask") (roundrect_rratio 0.2083333333)
       (net 7 "PV") (pinfunction "S") (pintype "passive"))
     (model "${KICAD6_3DMODEL_DIR}/Package_TO_SOT_SMD.3dshapes/TO-252-2.wrl"
@@
   (segment (start 235.815 96.51) (end 234.188 96.51) (width 0.25) (layer "F.Cu") (net 2))
   (segment (start 264.8185 172.593) (end 264.922 172.4895) (width 0.254) (layer "F.Cu") (net 4))
+  (via (at 279.4 172.72) (size 0.8) (drill 0.4) (layers "F.Cu" "B.Cu") (free) (net 4))
+  (via (at 257.81 172.72) (size 0.8) (drill 0.4) (layers "F.Cu" "B.Cu") (free) (net 4))
+  (via (at 237.49 172.72) (size 0.8) (drill 0.4) (layers "F.Cu" "B.Cu") (free) (net 4))
   (segment (start 273.2525 108.6115) (end 276.454 105.41) (width 0.25) (layer "F.Cu") (net 5))
   (segment (start 267.183 108.6115) (end 273.2525 108.6115) (width 0.25) (layer "F.Cu") (net 5))
