File: Reverse polarity breakout board/fuse breakout board/_autosave-fuse breakout board.kicad_sch (KiCad schematic)
At the start: 7 parts

Commit message: Reworked power planes and adjusted cap bank
Reworked power plane and adjusted cap bank. Created a 35 mill trace from heatsink die to pad off power plane to account for ground connection
Parts:
- Conn1: footprint MRDT_Connectors:Square_Anderson_1_H -> MRDT_Connectors:Square_Anderson_2_H_Side_By_Side_PV
- Conn1: footprint (none) -> MRDT_Connectors:Square_Anderson_2_H_Side_By_Side_PV
Changed lines of the file:
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@@
 			)
 		)
-		(property "Footprint" "MRDT_Connectors:Square_Anderson_1_H"
+		(property "Footprint" "MRDT_Connectors:Square_Anderson_2_H_Side_By_Side_PV"
 			(at 17.78 54.61 0)
 			(effects
@@
 			)
 		)
-		(property "Footprint" ""
+		(property "Footprint" "MRDT_Connectors:Square_Anderson_2_H_Side_By_Side_PV"
 			(at 17.78 67.31 0)
 			(effects
