File: Power_Management_2025_Rev1/Power_Management_2025_Rev1.kicad_pcb (KiCad board)
At the start: 2 copper layers, 103 parts, among them J1 RJ45_LED_Shielded, Q1 BSS138, Q2 IPB180N10S4-02, Q3 IPB180N10S4-02, Q4 IPB180N10S4-02, U1 Teensy4.1_DEV-16771, U10 LT1910, U11 LT1910, U12 PKE3316ZPI, U13 PKE3316ZPI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

Commit message: Started on PCB editor
Started layout grouped components began trace work
Parts:
- removed U7, U8, U9: ~, Package_SO:SOIC-8_3.9x4.9mm_P1.27mm
- Conn1, Conn19: footprint MRDT_Connectors:Anderson_1_Horizontal -> MRDT_Connectors:Square_Anderson_2_H_Side_By_Side_PV; moved to B.Cu
- Conn10, Conn11, Conn12, Conn13, Conn14, Conn15, Conn16, Conn17, Conn18: footprint MRDT_Connectors:Anderson_1_Horizontal -> MRDT_Connectors:Square_Anderson_2_H_Side_By_Side_PV
- Conn20: moved to B.Cu
- Conn4, Conn5, Conn6, Conn7, Conn8: footprint MRDT_Connectors:Square_Anderson_2_H_Stacked -> MRDT_Connectors:Square_Anderson_2_H_Side_By_Side_PV
- U4, U5, U6: value ~ -> Opamp_Dual; footprint Package_SO:SOIC-8_3.9x4.9mm_P1.27mm -> Package_SO:SO-8_3.9x4.9mm_P1.27mm
- moved C8 388.2 mm to (427.5, -87.0)
- moved R29 356.5 mm to (433.6, 266.0)
- moved R30 356.5 mm to (433.6, 268.5)
- moved R31 356.5 mm to (433.6, 271.0)
- moved R32 356.5 mm to (433.6, 273.5)
- moved R33 356.5 mm to (433.6, 276.0)
- moved R34 356.5 mm to (433.6, 278.5)
- moved R35 356.5 mm to (433.6, 281.0)
- moved U13 348.2 mm to (394.9, -99.1)
- moved Conn15 335.0 mm to (-180.2, -98.5)
- moved C10 332.8 mm to (341.0, -96.0)
- moved Conn14 321.3 mm to (-185.2, -74.0)
- moved D3 304.5 mm to (-0.14, -110.2)
- moved Q1 304.5 mm to (17.6, -110.0)
- moved Conn17 304.2 mm to (-183.6, -12.4)
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Connections:
- R10 pad 2: Net-(U4--) -> Net-(U6B--)
- R11 pad 1: Net-(U5-+) -> Net-(U4A-+)
- R12 pad 1: Net-(U5-+) -> Net-(U4A-+)
- R13 pad 1: Net-(U5--) -> Net-(U4A--)
- R14 pad 2: Net-(U5--) -> Net-(U4A--)
- R15 pad 1: Net-(U6-+) -> Net-(U4B-+)
- R16 pad 1: Net-(U6-+) -> Net-(U4B-+)
- R17 pad 1: Net-(U6--) -> Net-(U4B--)
- R18 pad 2: Net-(U6--) -> Net-(U4B--)
- R19 pad 1: Net-(U8-+) -> Net-(U5A-+)
- R20 pad 1: Net-(U8-+) -> Net-(U5A-+)
- R21 pad 1: Net-(U8--) -> Net-(U5A--)
- R22 pad 2: Net-(U8--) -> Net-(U5A--)
- R23 pad 1: Net-(U9-+) -> Net-(U5B-+)
- R24 pad 1: Net-(U9-+) -> Net-(U5B-+)
- R25 pad 1: Net-(U9--) -> Net-(U5B--)
- R26 pad 2: Net-(U9--) -> Net-(U5B--)
- R3 pad 1: Net-(U7--) -> Net-(U6A--)
- R4 pad 2: Net-(U7--) -> Net-(U6A--)
- R5 pad 1: Net-(U7-+) -> Net-(U6A-+)
- R6 pad 1: Net-(U7-+) -> Net-(U6A-+)
- R7 pad 1: Net-(U4-+) -> Net-(U6B-+)
- R8 pad 1: Net-(U4-+) -> Net-(U6B-+)
- R9 pad 1: Net-(U4--) -> Net-(U6B--)
- U1 pad 14: C_SENSE -> CURRENT_SENSE
- U4 pad 1: Net-(U4-+) -> CELL_SENSE_3
- U4 pad 2: Net-(U4--) -> Net-(U4A--)
- U4 pad 3: +BATT -> Net-(U4A-+)
- U4 pad 5: CELL_SENSE_2 -> Net-(U4B-+)
- U4 pad 6: (no net) -> Net-(U4B--)
- U4 pad 7: (no net) -> CELL_SENSE_4
- U4 pad 8: (no net) -> +BATT
- U5 pad 1: Net-(U5-+) -> CELL_SENSE_5
- U5 pad 2: Net-(U5--) -> Net-(U5A--)
- U5 pad 3: +BATT -> Net-(U5A-+)
- U5 pad 5: CELL_SENSE_3 -> Net-(U5B-+)
- U5 pad 6: (no net) -> Net-(U5B--)
- U5 pad 7: (no net) -> CELL_SENSE_6
- U5 pad 8: (no net) -> +BATT
- U6 pad 1: Net-(U6-+) -> CELL_SENSE_1
- U6 pad 2: Net-(U6--) -> Net-(U6A--)
- U6 pad 3: +BATT -> Net-(U6A-+)
- U6 pad 5: CELL_SENSE_4 -> Net-(U6B-+)
- U6 pad 6: (no net) -> Net-(U6B--)
- U6 pad 7: (no net) -> CELL_SENSE_2
- U6 pad 8: (no net) -> +BATT
Routing:
- net CELL_SENSE_2: track 0.00 -> 151.9 mm, vias 0 -> 4
- net CELL_SENSE_1: track 0.00 -> 141.4 mm, vias 0 -> 4
- net AUX_EN: track 0.00 -> 134.0 mm, vias 0 -> 4
- net LC_EN: track 0.00 -> 133.2 mm, vias 0 -> 3
- net CELL_SENSE_4: track 0.00 -> 115.0 mm, vias 0 -> 4
- net MOTOR_EN: track 0.00 -> 112.4 mm, vias 0 -> 3
- net +3.3V: track 0.00 -> 109.8 mm, vias 0 -> 1
- net CELL_SENSE_3: track 0.00 -> 109.3 mm, vias 0 -> 4
- net CELL_SENSE2_1: track 0.00 -> 90.3 mm, vias 0 -> 1
- net CURRENT_SENSE: track 0.00 -> 89.3 mm, vias 0 -> 1
- net CELL_SENSE_6: track 0.00 -> 76.2 mm, vias 0 -> 6
- net CELL_SENSE_5: track 0.00 -> 75.9 mm, vias 0 -> 4
- net CELL_SENSE2_2: track 0.00 -> 68.5 mm
- net CELL_SENSE2_3: track 0.00 -> 64.9 mm
- net CELL_SENSE2_4: track 0.00 -> 62.4 mm
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
Commit message: Tracing
made a few more traces with the buzzer and cap bank
Parts:
- moved R1 202.9 mm to (86.6, 58.5), turned to -90 degrees
- moved D3 192.2 mm to (90.3, 59.4), turned to 180 degrees
- moved B1 189.2 mm to (85.4, 49.7)
- moved Q1 186.2 mm to (94.6, 59.5), turned to 180 degrees
- moved F1 171.7 mm to (27.4, 135.0), turned to 90 degrees
- moved C4 152.4 mm to (24.4, 114.8), turned to 0 degrees
- moved C5 144.3 mm to (24.2, 96.3)
- moved D1 142.0 mm to (28.5, 39.2), turned to 90 degrees
- moved C6 138.5 mm to (23.9, 78.0)
- moved C7 136.9 mm to (23.9, 59.5)
- moved C2 29.6 mm to (144.5, -112.0), turned to -90 degrees
- moved C1 8.47 mm to (124.0, -112.0), turned to -90 degrees
Connections:
- U1 pad 22: BUZZER -> unconnected-(U1-A8-Pad22)
- U1 pad 39: unconnected-(U1-A15-Pad39) -> BUZZER
Routing:
- net Net-(D1-K): track 0.00 -> 87.1 mm
- net Net-(B1-V-): track 0.00 -> 12.5 mm
- net +3.3V: track 109.8 -> 118.2 mm
- net Net-(D3-A): track 0.00 -> 2.82 mm

Commit message: Adjusted components for power planes
Adjusted components for power planes and had the layout reviewed by E-Leads. Changes to follow
Parts:
- moved Conn10 432.9 mm to (289.2, -25.8), turned to -90 degrees
- moved Conn8 371.9 mm to (273.1, -25.9), turned to -90 degrees
- moved Conn7 353.0 mm to (257.0, -25.8), turned to -90 degrees
- moved Conn6 334.7 mm to (240.8, -25.8), turned to -90 degrees
- moved Conn5 317.7 mm to (224.7, -25.8), turned to -90 degrees
- moved Conn4 301.4 mm to (208.6, -25.8), turned to -90 degrees
- moved Conn17 300.2 mm to (108.9, -79.7)
- moved Conn14 297.4 mm to (109.0, -31.2)
- moved Conn11 293.7 mm to (154.0, -41.5)
- moved Conn12 293.7 mm to (152.4, -100.6)
- moved Conn13 293.7 mm to (154.0, -23.4)
- moved Conn15 293.6 mm to (108.9, -47.4)
- moved Conn18 280.8 mm to (108.9, -95.8)
- moved U3 268.2 mm to (3.69, 65.0)
- moved R29 262.9 mm to (234.7, 94.0)
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Routing:
- net Net-(D1-K): track 87.1 -> 0.72 mm

Commit message: Update Power_Management_2025_Rev1.kicad_pcb
Parts:
- moved C14 107.1 mm to (81.6, 36.6), turned to -90 degrees
- moved Q3 104.3 mm to (90.5, 34.6), turned to 90 degrees
- moved D6 98.0 mm to (161.1, 75.5)
- moved Q2 97.7 mm to (108.7, 34.5), turned to 90 degrees
- moved Q4 97.5 mm to (126.5, 34.5), turned to 90 degrees
- moved C12 97.0 mm to (99.6, 36.9), turned to -90 degrees
- moved C9 93.7 mm to (117.6, 36.6), turned to -90 degrees
- moved D10 92.9 mm to (164.5, 125.4)
- moved D5 92.9 mm to (164.5, 112.4)
- moved D7 92.9 mm to (164.5, 117.6)
- moved D8 92.9 mm to (164.5, 120.2)
- moved D9 92.9 mm to (164.5, 122.8)
- moved R31 83.0 mm to (155.1, 75.5)
- moved R30 80.9 mm to (155.4, 112.5)
- moved R32 80.9 mm to (155.4, 117.5)
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Routing:
- net NS_24V: track 0.00 -> 105.8 mm, vias 0 -> 3
- net MOTOR_EN: track 112.4 -> 47.0 mm, vias 3 -> 4
- net AUX_EN: track 134.0 -> 69.0 mm, vias 4 -> 5
- net LC_EN: track 133.2 -> 69.3 mm, vias 3 -> 4
- net +3.3V: track 118.2 -> 128.8 mm, vias 1 -> 3
- net +5V: track 19.1 -> 16.6 mm, vias 3 -> 0
- net Net-(Q3-G): track 14.7 -> 17.2 mm

Commit message: More tracework
Made corrections to schematic and did more tracework on PCB
Parts:
- moved Conn18 200.0 mm to (268.1, 25.2), turned to -90 degrees
- moved Conn4 180.6 mm to (35.2, 24.7)
- moved Conn5 178.4 mm to (53.8, 25.2)
- moved D5 178.0 mm to (336.9, 68.4)
- moved D7 178.0 mm to (336.9, 73.6)
- moved D8 178.0 mm to (336.9, 76.2)
- moved D9 178.0 mm to (336.9, 78.7)
- moved R30 178.0 mm to (327.9, 68.5)
- moved R32 178.0 mm to (327.9, 73.5)
- moved R33 178.0 mm to (327.9, 76.0)
- moved R34 178.0 mm to (327.9, 78.5)
- moved Conn17 177.4 mm to (252.0, 25.2), turned to -90 degrees
- moved Conn6 175.6 mm to (72.8, 25.3)
- moved Conn7 173.2 mm to (91.6, 25.7)
- moved Conn8 172.7 mm to (108.1, 25.2)
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Connections:
- C1 pad 1: +BATT -> IP-
- C12 pad 1: +BATT -> IP-
- C14 pad 1: +BATT -> IP-
- C4 pad 1: Net-(D1-K) -> IP+
- C5 pad 1: Net-(D1-K) -> IP+
- C6 pad 1: Net-(D1-K) -> IP+
- C7 pad 1: Net-(D1-K) -> IP+
- C9 pad 1: +BATT -> IP-
- D1 pad 1: Net-(D1-K) -> IP+
- F1 pad 1: +BATT -> IP-
- F1 pad 2: Net-(D1-K) -> IP+
- Q2 pad 4: +BATT -> IP-
- Q3 pad 4: +BATT -> IP-
- Q4 pad 4: +BATT -> IP-
- R2 pad 1: +5V -> FF_AUX
- R27 pad 1: +5V -> FF_LC
- R28 pad 1: +5V -> FF_MOTOR
- R35 pad 1: +BATT -> IP-
- U1 pad 22: unconnected-(U1-A8-Pad22) -> FF_MOTOR
- U1 pad 40: unconnected-(U1-A16-Pad40) -> FF_LC
- U1 pad 41: ESTOP -> FF_AUX
- U10 pad 6: +BATT -> IP-
- U10 pad 8: +BATT -> IP-
- U11 pad 6: +BATT -> IP-
- U11 pad 8: +BATT -> IP-
- U12 pad 3: +BATT -> IP-
- U13 pad 3: +BATT -> IP-
- U14 pad 6: +BATT -> IP-
- U14 pad 8: +BATT -> IP-
- U2 pad 1: +BATT -> IP-
- U3 pad 3: C_SENSE -> CURRENT_SENSE
- U3 pad 4: +BATT -> IP+
- U3 pad 5: PACK_OUT -> IP-
- U4 pad 8: +BATT -> IP-
- U5 pad 8: +BATT -> IP-
- U6 pad 8: +BATT -> IP-
Routing:
- net NS_ENABLE: track 0.00 -> 165.7 mm, vias 0 -> 1
- net Net-(U10-FAULT): track 3.19 -> 156.0 mm, vias 0 -> 2
- net POE_ENABLE: track 0.00 -> 137.0 mm, vias 0 -> 1
- net LC_EN: track 69.3 -> 182.7 mm, vias 4 -> 3
- net NS_24V: track 105.8 -> 0.00 mm, vias 3 -> 0
- net FF_MOTOR: track 0.00 -> 74.0 mm, vias 0 -> 2
- net FF_AUX: track 0.00 -> 41.9 mm, vias 0 -> 2
- net FF_LC: track 0.00 -> 37.2 mm, vias 0 -> 2
- net Net-(U14-FAULT): track 3.75 -> 40.5 mm, vias 0 -> 2
- net AUX_EN: track 69.0 -> 92.1 mm, vias 5 -> 4
- net +5V: track 16.6 -> 0.00 mm
- net IP+: track 0.00 -> 10.9 mm
- net Net-(Q2-G): track 13.0 -> 19.6 mm
- net Net-(Q3-G): track 17.2 -> 21.9 mm
- net Net-(Q4-G): track 20.6 -> 19.0 mm
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
Commit message: Rearranged component
We Made power planes
Parts:
- C1, C11, C12, C13, C14, C2, C9: footprint Capacitor_THT:CP_Radial_D5.0mm_P2.00mm -> Capacitor_SMD:C_1206_3216Metric_Pad1.33x1.80mm_HandSolder
- C10, C8: footprint Capacitor_THT:CP_Radial_Tantal_D5.0mm_P5.00mm -> Capacitor_THT:CP_Radial_D5.0mm_P2.00mm
- R10, R11, R14, R15, R18, R19, R22, R23, R26, R4, R6, R7: value 36.5k -> 39k
- R12, R13, R16, R17, R20, R21, R24, R25, R3, R5, R8, R9: value 46.4k -> 47k
- moved R32 258.1 mm to (74.1, 26.5)
- moved D7 252.5 mm to (85.3, 52.8)
- moved D4 181.3 mm to (118.9, 41.0)
- moved R29 181.3 mm to (111.8, 41.0)
- moved D5 179.8 mm to (172.6, 141.2)
- moved R30 175.4 mm to (168.3, 141.2)
- moved D8 171.5 mm to (165.7, 68.3)
- moved R33 171.1 mm to (157.0, 68.3)
- moved D9 170.0 mm to (167.0, 82.0)
- moved R34 170.0 mm to (157.9, 81.8)
- moved C1 167.1 mm to (104.0, 49.9)
- moved C2 166.4 mm to (124.5, 52.0), turned to 0 degrees
- moved U2 160.7 mm to (116.6, 54.0), turned to 90 degrees
- moved Conn12 118.4 mm to (209.5, 140.9), turned to 180 degrees
- moved U13 109.7 mm to (177.9, 160.6), turned to 90 degrees
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Connections:
- Conn1 pad 4: +BATT -> IP+
- Conn19 pad 4: +BATT -> IP+
Routing:
- net Net-(U10-FAULT): track 156.0 -> 3.20 mm, vias 2 -> 0
- net LC_EN: track 182.7 -> 47.7 mm, vias 3 -> 1
- net CURRENT_SENSE: track 89.3 -> 199.4 mm, vias 1 -> 7
- net NS_ENABLE: track 165.7 -> 64.6 mm, vias 1 -> 2
- net POE_ENABLE: track 137.0 -> 94.6 mm, vias 1 -> 2
- net Net-(Q2-G): track 19.6 -> 0.00 mm
- net Net-(Q3-G): track 21.9 -> 33.4 mm
- net +3.3V: track 127.8 -> 117.5 mm, vias 2 -> 1
- net LOW_CURRENT_PWR: track 6.35 -> 0.00 mm
- net CELL_SENSE_6: track 76.2 -> 78.0 mm
- net CELL_SENSE_5: track 75.9 -> 77.7 mm
- net CELL_SENSE_4: track 115.0 -> 116.8 mm
- net CELL_SENSE_3: track 109.3 -> 111.1 mm
- net CELL_SENSE_2: track 151.9 -> 153.7 mm
- net CELL_SENSE_1: track 141.4 -> 143.2 mm
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- added copper zone on F.Cu, net AUX_PWR
- added copper zone on B.Cu, net GND
- added copper zone on F.Cu, net GND
- added copper zone on F.Cu, net IP+
- added copper zone on F.Cu, net IP-
- added copper zone on F.Cu, net LOW_CURRENT_PWR
- added copper zone on F.Cu, net MOTOR_PWR
- added copper zone on F.Cu, net NS_24V
- added copper zone on F.Cu, net POE_24V
Other:
- board text added: "NS PWR"
- board text added: "POE PWR"

Commit message: Finished Rev 1 Design for CDR
Organized components, laid power planes, ran traces, and finished board edge cuts
Parts:
- Conn1: moved to F.Cu
- U10, U11, U14: footprint Package_SO:SOIC-8-N7_3.9x4.9mm_P1.27mm -> Package_SO:SOIC-8_3.9x4.9mm_P1.27mm
- moved R27 105.5 mm to (204.2, 78.0), turned to 180 degrees
- moved D4 85.3 mm to (43.8, 81.6), turned to -90 degrees
- moved R29 81.5 mm to (43.8, 85.9), turned to 90 degrees
- moved R2 78.0 mm to (179.3, 92.4), turned to 90 degrees
- moved C9 66.7 mm to (67.1, 69.0), turned to 180 degrees
- moved C2 65.7 mm to (170.9, 98.5), turned to -90 degrees
- moved U2 63.9 mm to (170.9, 87.7), turned to -90 degrees
- moved D3 57.0 mm to (176.0, 119.5)
- moved Q1 57.0 mm to (180.2, 119.5)
- moved B1 57.0 mm to (171.1, 109.8)
- moved R1 57.0 mm to (172.3, 118.6)
- moved C10 55.9 mm to (211.4, 121.6)
- moved H2 51.3 mm to (231.8, 183.4)
- moved R34 51.1 mm to (206.8, 66.6), turned to -90 degrees
- moved R31 47.9 mm to (204.7, 119.7)
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Routing:
- net +3.3V: track 117.5 -> 324.2 mm, vias 1 -> 6
- net IP-: track 0.00 -> 206.1 mm, vias 0 -> 8
- net LOW_CURRENT_PWR: track 0.00 -> 102.4 mm
- net FF_LC: track 37.2 -> 126.9 mm, vias 2 -> 4
- net RX-: track 0.00 -> 78.8 mm, vias 0 -> 1
- net LED: track 0.00 -> 78.5 mm, vias 0 -> 2
- net BUZZER: track 0.00 -> 78.1 mm, vias 0 -> 1
- net LC_EN: track 47.7 -> 125.4 mm, vias 1 -> 4
- net RX+: track 0.00 -> 77.3 mm, vias 0 -> 1
- net TX+: track 0.00 -> 71.2 mm, vias 0 -> 1
- net TX-: track 0.00 -> 70.9 mm, vias 0 -> 1
- net AUX_EN: track 92.1 -> 152.9 mm
- net NS_24V: track 0.00 -> 55.4 mm
- net FF_AUX: track 41.9 -> 86.8 mm, vias 2 -> 3
- net POE_24V: track 0.00 -> 40.9 mm
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- removed copper zone on F.Cu, net LOW_CURRENT_PWR
- removed copper zone on F.Cu, net NS_24V
- removed copper zone on F.Cu, net POE_24V
Other:
- board outline added: 213.1 x 179.3 mm
- board text added: "+3.3V"
- board text added: "AUX PWR"
- board text added: "LC PORT"
- board text added: "LC PWR"
- board text added: "MOTOR PORT"
- board text added: "MOTOR PWR"
- board text added: "NS PORT"
- board text added: "PMS 2025 Rev 1 Mars Rover Design Team Ethan Coggshell, Luke Duff, Sean Duda"
- board text added: "POE PORT"
- board text added: "PV+"
