File: board/Voltage_Sensing.kicad_sch (KiCad schematic)
At the start: 41 parts, among them U18 Opamp_Dual, U4 Opamp_Dual, U5 Opamp_Dual, U6 Opamp_Dual

Commit message: Changed footprints to handsolder version
Parts:
- R10, R11, R12, R13, R14, R15, R16, R17, R18, R19, R20, R21, R22, R23, R24, R25, R26, R28, R29, R30, R31, R32, R33, R4, R40, R5, R6, R7, R8, R9: footprint Resistor_SMD:R_0603_1608Metric -> Resistor_SMD:R_0603_1608Metric_Pad0.98x0.95mm_HandSolder
Changed lines of the file:
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@@
 			)
 		)
-		(property "Footprint" "Resistor_SMD:R_0603_1608Metric"
+		(property "Footprint" "Resistor_SMD:R_0603_1608Metric_Pad0.98x0.95mm_HandSolder"
 			(at 143.256 46.736 90)
 			(effects
@@
 			)
 		)
-		(property "Footprint" "Resistor_SMD:R_0603_1608Metric"
+		(property "Footprint" "Resistor_SMD:R_0603_1608Metric_Pad0.98x0.95mm_HandSolder"
 			(at 138.176 110.236 90)
 			(effects
@@
 			)
 		)
-		(property "Footprint" "Resistor_SMD:R_0603_1608Metric"
+		(property "Footprint" "Resistor_SMD:R_0603_1608Metric_Pad0.98x0.95mm_HandSolder"
 			(at 171.704 110.744 90)
 			(effects
@@
 			)
 		)
-		(property "Footprint" "Resistor_SMD:R_0603_1608Metric"
+		(property "Footprint" "Resistor_SMD:R_0603_1608Metric_Pad0.98x0.95mm_HandSolder"
 			(at 152.146 140.716 90)
 			(effects
@@
 			)
 		)
-		(property "Footprint" "Resistor_SMD:R_0603_1608Metric"
+		(property "Footprint" "Resistor_SMD:R_0603_1608Metric_Pad0.98x0.95mm_HandSolder"
 			(at 153.416 122.936 90)
 			(effects
@@
 			)
 		)
-		(property "Footprint" "Resistor_SMD:R_0603_1608Metric"
+		(property "Footprint" "Resistor_SMD:R_0603_1608Metric_Pad0.98x0.95mm_HandSolder"
 			(at 143.256 35.306 90)
 			(effects
@@
 			)
 		)
-		(property "Footprint" "Resistor_SMD:R_0603_1608Metric"
+		(property "Footprint" "Resistor_SMD:R_0603_1608Metric_Pad0.98x0.95mm_HandSolder"
 			(at 175.514 56.134 90)
 			(effects
@@
 			)
 		)
-		(property "Footprint" "Resistor_SMD:R_0603_1608Metric"
+		(property "Footprint" "Resistor_SMD:R_0603_1608Metric_Pad0.98x0.95mm_HandSolder"
 			(at 143.256 40.386 90)
 			(effects
@@
 			)
 		)
-		(property "Footprint" "Resistor_SMD:R_0603_1608Metric"
+		(property "Footprint" "Resistor_SMD:R_0603_1608Metric_Pad0.98x0.95mm_HandSolder"
 			(at 155.956 86.106 90)
 			(effects
@@
 			)
 		)
-		(property "Footprint" "Resistor_SMD:R_0603_1608Metric"
+		(property "Footprint" "Resistor_SMD:R_0603_1608Metric_Pad0.98x0.95mm_HandSolder"
 			(at 141.986 64.516 90)
 			(effects
@@
 			)
 		)
-		(property "Footprint" "Resistor_SMD:R_0603_1608Metric"
+		(property "Footprint" "Resistor_SMD:R_0603_1608Metric_Pad0.98x0.95mm_HandSolder"
 			(at 140.716 78.486 90)
 			(effects
@@
 			)
 		)
-		(property "Footprint" "Resistor_SMD:R_0603_1608Metric"
+		(property "Footprint" "Resistor_SMD:R_0603_1608Metric_Pad0.98x0.95mm_HandSolder"
 			(at 157.226 68.326 90)
 			(effects
@@
 			)
 		)
-		(property "Footprint" "Resistor_SMD:R_0603_1608Metric"
+		(property "Footprint" "Resistor_SMD:R_0603_1608Metric_Pad0.98x0.95mm_HandSolder"
 			(at 136.906 128.016 90)
 			(effects
@@
 			)
 		)
-		(property "Footprint" "Resistor_SMD:R_0603_1608Metric"
+		(property "Footprint" "Resistor_SMD:R_0603_1608Metric_Pad0.98x0.95mm_HandSolder"
 			(at 139.446 101.346 90)
 			(effects
@@
 			)
 		)
-		(property "Footprint" "Resistor_SMD:R_0603_1608Metric"
+		(property "Footprint" "Resistor_SMD:R_0603_1608Metric_Pad0.98x0.95mm_HandSolder"
 			(at 138.176 119.126 90)
 			(effects
@@
 			)
 		)
-		(property "Footprint" "Resistor_SMD:R_0603_1608Metric"
+		(property "Footprint" "Resistor_SMD:R_0603_1608Metric_Pad0.98x0.95mm_HandSolder"
 			(at 140.716 83.566 90)
 			(effects
@@
 			)
 		)
-		(property "Footprint" "Resistor_SMD:R_0603_1608Metric"
+		(property "Footprint" "Resistor_SMD:R_0603_1608Metric_Pad0.98x0.95mm_HandSolder"
 			(at 140.716 73.406 90)
 			(effects
@@
 			)
 		)
-		(property "Footprint" "Resistor_SMD:R_0603_1608Metric"
+		(property "Footprint" "Resistor_SMD:R_0603_1608Metric_Pad0.98x0.95mm_HandSolder"
 			(at 174.244 73.914 90)
 			(effects
@@
 			)
 		)
-		(property "Footprint" "Resistor_SMD:R_0603_1608Metric"
+		(property "Footprint" "Resistor_SMD:R_0603_1608Metric_Pad0.98x0.95mm_HandSolder"
 			(at 138.176 115.316 90)
 			(effects
@@
 			)
 		)
-		(property "Footprint" "Resistor_SMD:R_0603_1608Metric"
+		(property "Footprint" "Resistor_SMD:R_0603_1608Metric_Pad0.98x0.95mm_HandSolder"
 			(at 170.434 128.524 90)
 			(effects
@@
 			)
 		)
-		(property "Footprint" "Resistor_SMD:R_0603_1608Metric"
+		(property "Footprint" "Resistor_SMD:R_0603_1608Metric_Pad0.98x0.95mm_HandSolder"
 			(at 139.446 92.456 90)
 			(effects
@@
 			)
 		)
-		(property "Footprint" "Resistor_SMD:R_0603_1608Metric"
+		(property "Footprint" "Resistor_SMD:R_0603_1608Metric_Pad0.98x0.95mm_HandSolder"
 			(at 144.526 26.416 90)
 			(effects
@@
 			)
 		)
-		(property "Footprint" "Resistor_SMD:R_0603_1608Metric"
+		(property "Footprint" "Resistor_SMD:R_0603_1608Metric_Pad0.98x0.95mm_HandSolder"
 			(at 141.986 60.706 90)
 			(effects
@@
 			)
 		)
-		(property "Footprint" "Resistor_SMD:R_0603_1608Metric"
+		(property "Footprint" "Resistor_SMD:R_0603_1608Metric_Pad0.98x0.95mm_HandSolder"
 			(at 136.906 133.096 90)
 			(effects
@@
 			)
 		)
-		(property "Footprint" "Resistor_SMD:R_0603_1608Metric"
+		(property "Footprint" "Resistor_SMD:R_0603_1608Metric_Pad0.98x0.95mm_HandSolder"
 			(at 172.974 92.964 90)
 			(effects
@@
 			)
 		)
-		(property "Footprint" "Resistor_SMD:R_0603_1608Metric"
+		(property "Footprint" "Resistor_SMD:R_0603_1608Metric_Pad0.98x0.95mm_HandSolder"
 			(at 158.496 48.006 90)
 			(effects
@@
 			)
 		)
-		(property "Footprint" "Resistor_SMD:R_0603_1608Metric"
+		(property "Footprint" "Resistor_SMD:R_0603_1608Metric_Pad0.98x0.95mm_HandSolder"
 			(at 141.986 55.626 90)
 			(effects
@@
 			)
 		)
-		(property "Footprint" "Resistor_SMD:R_0603_1608Metric"
+		(property "Footprint" "Resistor_SMD:R_0603_1608Metric_Pad0.98x0.95mm_HandSolder"
 			(at 154.686 105.156 90)
 			(effects
@@
 			)
 		)
-		(property "Footprint" "Resistor_SMD:R_0603_1608Metric"
+		(property "Footprint" "Resistor_SMD:R_0603_1608Metric_Pad0.98x0.95mm_HandSolder"
 			(at 139.446 97.536 90)
 			(effects
@@
 			)
 		)
-		(property "Footprint" "Resistor_SMD:R_0603_1608Metric"
+		(property "Footprint" "Resistor_SMD:R_0603_1608Metric_Pad0.98x0.95mm_HandSolder"
 			(at 176.784 35.814 90)
 			(effects

Commit message: fixed op amp footprint
Parts:
- U18, U4, U5, U6: footprint KiCad:SOIC127P600X175-8N -> PowerManagementBoard:SOIC127P600X175-8N
Changed lines of the file:
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@@
 			)
 		)
-		(property "Footprint" "KiCad:SOIC127P600X175-8N"
+		(property "Footprint" "PowerManagementBoard:SOIC127P600X175-8N"
 			(at 153.67 93.98 0)
 			(effects
@@
 			)
 		)
-		(property "Footprint" "KiCad:SOIC127P600X175-8N"
+		(property "Footprint" "PowerManagementBoard:SOIC127P600X175-8N"
 			(at 151.13 129.54 0)
 			(effects
@@
 			)
 		)
-		(property "Footprint" "KiCad:SOIC127P600X175-8N"
+		(property "Footprint" "PowerManagementBoard:SOIC127P600X175-8N"
 			(at 152.4 111.76 0)
 			(effects
@@
 			)
 		)
-		(property "Footprint" "KiCad:SOIC127P600X175-8N"
+		(property "Footprint" "PowerManagementBoard:SOIC127P600X175-8N"
 			(at 214.63 45.72 0)
 			(effects
@@
 			)
 		)
-		(property "Footprint" "KiCad:SOIC127P600X175-8N"
+		(property "Footprint" "PowerManagementBoard:SOIC127P600X175-8N"
 			(at 245.11 46.99 0)
 			(effects
@@
 			)
 		)
-		(property "Footprint" "KiCad:SOIC127P600X175-8N"
+		(property "Footprint" "PowerManagementBoard:SOIC127P600X175-8N"
 			(at 154.94 74.93 0)
 			(effects
@@
 			)
 		)
-		(property "Footprint" "KiCad:SOIC127P600X175-8N"
+		(property "Footprint" "PowerManagementBoard:SOIC127P600X175-8N"
 			(at 157.48 36.83 0)
 			(effects
@@
 			)
 		)
-		(property "Footprint" "KiCad:SOIC127P600X175-8N"
+		(property "Footprint" "PowerManagementBoard:SOIC127P600X175-8N"
 			(at 229.87 45.72 0)
 			(effects
@@
 			)
 		)
-		(property "Footprint" "KiCad:SOIC127P600X175-8N"
+		(property "Footprint" "PowerManagementBoard:SOIC127P600X175-8N"
 			(at 156.21 57.15 0)
 			(effects

Commit message: designated an area for each circuit on pcb
Parts:
- renumbered U18 to U5
Changed lines of the file:
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@@
 		(dnp no)
 		(fields_autoplaced yes)
-		(property "Reference" "U18"
+		(property "Reference" "U5"
 			(at 157.48 26.67 0)
 			(effects
@@
 			(project ""
 				(path "/7eaa639d-7062-45e7-be05-1c2855431307/77b38e11-7bca-4b0d-9192-77b02a5f3429"
-					(reference "U18")
+					(reference "U5")
 					(unit 1)
 				)

Commit message: Configuration of parts
Parts:
- Conn1: footprint MRDT_Connectors:MOLEX_SL_07_Horizontal -> MRDT_Connectors:MOLEX_SL_07_Vertical
Changed lines of the file:
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@@
 		(on_board yes)
 		(dnp no)
-		(fields_autoplaced yes)
 		(property "Reference" "U6"
 			(at 152.4 101.6 0)
@@
 		)
 		(property "Value" "Opamp_Dual"
-			(at 152.4 104.14 0)
+			(at 160.528 109.474 0)
 			(effects
 				(font
@@
 			)
 		)
-		(property "Footprint" "MRDT_Connectors:MOLEX_SL_07_Horizontal"
+		(property "Footprint" "MRDT_Connectors:MOLEX_SL_07_Vertical"
 			(at 88.9 109.22 0)
 			(effects

Commit message: experimented with layout
Connections:
- net at R4.1, R6.1: now also U4.3 (+); no longer U4.5 (+)
- net at R30.1, R32.1: now also U6.5 (+); no longer U6.3 (+)
- net at R19.1, R21.1: now also U5.3 (+); no longer U5.5 (+)
- net at R20.1, R22.2: now also U5.2 (-); no longer U5.6 (-)
- net at R22.1, R29.1: now also U5.1; no longer U5.7
- net at R33.1, R40.1: now also U6.7; no longer U6.1
- net at R12.1, R13.1: now also U6.1; no longer U6.7
- net at R10.1, R12.2: now also U6.2 (-); no longer U6.6 (-)
- net at R31.1, R33.2: now also U6.6 (-); no longer U6.2 (-)
- net at R11.1, R9.1: now also U6.3 (+); no longer U6.5 (+)
- net at R24.1, R26.1: now also U4.5 (+); no longer U5.3 (+)
- net at R7.1, R8.1: now also U4.1; no longer U4.7
- net at R23.1, R25.2: now also U4.6 (-); no longer U5.2 (-)
- net at R17.1, R18.1: now also U5.7; no longer U4.1
- net at R15.1, R17.2: now also U5.6 (-); no longer U4.2 (-)
- net at R14.1, R16.1: now also U5.5 (+); no longer U4.3 (+)
- net at R5.1, R7.2: now also U4.2 (-); no longer U4.6 (-)
- net at R25.1, R28.1: now also U4.7; no longer U5.1
Other:
- moved on the sheet: U4A, U4B, U5A, U5B, U6A, U6B
Changed lines of the file:
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@@
 	(symbol
 		(lib_id "Device:Opamp_Dual")
-		(at 153.67 93.98 0)
+		(at 154.94 74.93 0)
 		(unit 2)
 		(exclude_from_sim no)
@@
 		(fields_autoplaced yes)
 		(property "Reference" "U5"
-			(at 153.67 83.82 0)
+			(at 154.94 64.77 0)
 			(effects
 				(font
@@
 		)
 		(property "Value" "Opamp_Dual"
-			(at 153.67 86.36 0)
+			(at 154.94 67.31 0)
 			(effects
 				(font
@@
 		)
 		(property "Footprint" "PowerManagementBoard:SOIC127P600X175-8N"
-			(at 153.67 93.98 0)
+			(at 154.94 74.93 0)
 			(effects
 				(font
@@
 		)
 		(property "Datasheet" "https://4donline.ihs.com/images/VipMasterIC/IC/DIOD/DIOD-S-A0005046231/DIOD-S-A0005046231-1.pdf?hkey=6D3A4C79FDBF58556ACFDE234799DDF0"
-			(at 153.67 93.98 0)
+			(at 154.94 74.93 0)
 			(effects
 				(font
@@
 		)
 		(property "Description" "Dual operational amplifier"
-			(at 153.67 93.98 0)
+			(at 154.94 74.93 0)
 			(effects
 				(font
@@
 		)
 		(property "Sim.Library" "${KICAD9_SYMBOL_DIR}/Simulation_SPICE.sp"
-			(at 153.67 93.98 0)
+			(at 154.94 74.93 0)
 			(effects
 				(font
@@
 		)
 		(property "Sim.Name" "kicad_builtin_opamp_dual"
-			(at 153.67 93.98 0)
+			(at 154.94 74.93 0)
 			(effects
 				(font
@@
 		)
 		(property "Sim.Device" "SUBCKT"
-			(at 153.67 93.98 0)
+			(at 154.94 74.93 0)
 			(effects
 				(font
@@
 		)
 		(property "Sim.Pins" "1=out1 2=in1- 3=in1+ 4=vee 5=in2+ 6=in2- 7=out2 8=vcc"
-			(at 153.67 93.98 0)
+			(at 154.94 74.93 0)
 			(effects
 				(font
@@
 	(symbol
 		(lib_id "Device:Opamp_Dual")
-		(at 151.13 129.54 0)
+		(at 152.4 111.76 0)
 		(unit 2)
 		(exclude_from_sim no)
@@
 		(on_board yes)
 		(dnp no)
-		(fields_autoplaced yes)
 		(property "Reference" "U6"
-			(at 151.13 119.38 0)
+			(at 152.4 101.6 0)
 			(effects
 				(font
@@
 		)
 		(property "Value" "Opamp_Dual"
-			(at 151.13 121.92 0)
+			(at 162.306 107.188 0)
 			(effects
 				(font
@@
 		)
 		(property "Footprint" "PowerManagementBoard:SOIC127P600X175-8N"
-			(at 151.13 129.54 0)
+			(at 152.4 111.76 0)
 			(effects
 				(font
@@
 		)
 		(property "Datasheet" "https://4donline.ihs.com/images/VipMasterIC/IC/DIOD/DIOD-S-A0005046231/DIOD-S-A0005046231-1.pdf?hkey=6D3A4C79FDBF58556ACFDE234799DDF0"
-			(at 151.13 129.54 0)
+			(at 152.4 111.76 0)
 			(effects
 				(font
@@
 		)
 		(property "Description" "Dual operational amplifier"
-			(at 151.13 129.54 0)
+			(at 152.4 111.76 0)
 			(effects
 				(font
@@
 		)
 		(property "Sim.Library" "${KICAD9_SYMBOL_DIR}/Simulation_SPICE.sp"
-			(at 151.13 129.54 0)
+			(at 152.4 111.76 0)
 			(effects
 				(font
@@
 		)
 		(property "Sim.Name" "kicad_builtin_opamp_dual"
-			(at 151.13 129.54 0)
+			(at 152.4 111.76 0)
 			(effects
 				(font
@@
 		)
 		(property "Sim.Device" "SUBCKT"
-			(at 151.13 129.54 0)
+			(at 152.4 111.76 0)
 			(effects
 				(font
@@
 		)
 		(property "Sim.Pins" "1=out1 2=in1- 3=in1+ 4=vee 5=in2+ 6=in2- 7=out2 8=vcc"
-			(at 151.13 129.54 0)
+			(at 152.4 111.76 0)
 			(effects
 				(font
@@
 	(symbol
 		(lib_id "Device:Opamp_Dual")
-		(at 152.4 111.76 0)
+		(at 151.13 129.54 0)
 		(unit 1)
 		(exclude_from_sim no)
@@
 		(dnp no)
 		(property "Reference" "U6"
-			(at 152.4 101.6 0)
+			(at 151.13 119.38 0)
 			(effects
 				(font
@@
 		)
 		(property "Value" "Opamp_Dual"
-			(at 160.528 109.474 0)
+			(at 159.258 127.254 0)
 			(effects
 				(font
@@
 		)
 		(property "Footprint" "PowerManagementBoard:SOIC127P600X175-8N"
-			(at 152.4 111.76 0)
+			(at 151.13 129.54 0)
 			(effects
 				(font
@@
 		)
 		(property "Datasheet" "https://4donline.ihs.com/images/VipMasterIC/IC/DIOD/DIOD-S-A0005046231/DIOD-S-A0005046231-1.pdf?hkey=6D3A4C79FDBF58556ACFDE234799DDF0"
-			(at 152.4 111.76 0)
+			(at 151.13 129.54 0)
 			(effects
 				(font
@@
 		)
 		(property "Description" "Dual operational amplifier"
-			(at 152.4 111.76 0)
+			(at 151.13 129.54 0)
 			(effects
 				(font
@@
 		)
 		(property "Sim.Library" "${KICAD9_SYMBOL_DIR}/Simulation_SPICE.sp"
-			(at 152.4 111.76 0)
+			(at 151.13 129.54 0)
 			(effects
 				(font
@@
 		)
 		(property "Sim.Name" "kicad_builtin_opamp_dual"
-			(at 152.4 111.76 0)
+			(at 151.13 129.54 0)
 			(effects
 				(font
@@
 		)
 		(property "Sim.Device" "SUBCKT"
-			(at 152.4 111.76 0)
+			(at 151.13 129.54 0)
 			(effects
 				(font
@@
 		)
 		(property "Sim.Pins" "1=out1 2=in1- 3=in1+ 4=vee 5=in2+ 6=in2- 7=out2 8=vcc"
-			(at 152.4 111.76 0)
+			(at 151.13 129.54 0)
 			(effects
 				(font
@@
 	(symbol
 		(lib_id "Device:Opamp_Dual")
-		(at 154.94 74.93 0)
+		(at 156.21 57.15 0)
 		(unit 1)
 		(exclude_from_sim no)
@@
 		(fields_autoplaced yes)
 		(property "Reference" "U4"
-			(at 154.94 64.77 0)
+			(at 156.21 46.99 0)
 			(effects
 				(font
@@
 		)
 		(property "Value" "Opamp_Dual"
-			(at 154.94 67.31 0)
+			(at 156.21 49.53 0)
 			(effects
 				(font
@@
 		)
 		(property "Footprint" "PowerManagementBoard:SOIC127P600X175-8N"
-			(at 154.94 74.93 0)
+			(at 156.21 57.15 0)
 			(effects
 				(font
@@
 		)
 		(property "Datasheet" "https://4donline.ihs.com/images/VipMasterIC/IC/DIOD/DIOD-S-A0005046231/DIOD-S-A0005046231-1.pdf?hkey=6D3A4C79FDBF58556ACFDE234799DDF0"
-			(at 154.94 74.93 0)
+			(at 156.21 57.15 0)
 			(effects
 				(font
@@
 		)
 		(property "Description" "Dual operational amplifier"
-			(at 154.94 74.93 0)
+			(at 156.21 57.15 0)
 			(effects
 				(font
@@
 		)
 		(property "Sim.Library" "${KICAD9_SYMBOL_DIR}/Simulation_SPICE.sp"
-			(at 154.94 74.93 0)
+			(at 156.21 57.15 0)
 			(effects
 				(font
@@
 		)
 		(property "Sim.Name" "kicad_builtin_opamp_dual"
-			(at 154.94 74.93 0)
+			(at 156.21 57.15 0)
 			(effects
 				(font
@@
 		)
 		(property "Sim.Device" "SUBCKT"
-			(at 154.94 74.93 0)
+			(at 156.21 57.15 0)
 			(effects
 				(font
@@
 		)
 		(property "Sim.Pins" "1=out1 2=in1- 3=in1+ 4=vee 5=in2+ 6=in2- 7=out2 8=vcc"
-			(at 154.94 74.93 0)
+			(at 156.21 57.15 0)
 			(effects
 				(font
@@
 	(symbol
 		(lib_id "Device:Opamp_Dual")
-		(at 157.48 36.83 0)
+		(at 153.67 93.98 0)
 		(unit 1)
 		(exclude_from_sim no)
@@
 		(on_board yes)
 		(dnp no)
-		(fields_autoplaced yes)
 		(property "Reference" "U5"
-			(at 157.48 26.67 0)
+			(at 153.67 83.82 0)
 			(effects
 				(font
@@
 		)
 		(property "Value" "Opamp_Dual"
-			(at 157.48 29.21 0)
+			(at 160.528 90.932 0)
 			(effects
 				(font
@@
 		)
 		(property "Footprint" "PowerManagementBoard:SOIC127P600X175-8N"
-			(at 157.48 36.83 0)
+			(at 153.67 93.98 0)
 			(effects
 				(font
@@
 		)
 		(property "Datasheet" "https://4donline.ihs.com/images/VipMasterIC/IC/DIOD/DIOD-S-A0005046231/DIOD-S-A0005046231-1.pdf?hkey=6D3A4C79FDBF58556ACFDE234799DDF0"
-			(at 157.48 36.83 0)
+			(at 153.67 93.98 0)
 			(effects
 				(font
@@
 		)
 		(property "Description" "Dual operational amplifier"
-			(at 157.48 36.83 0)
+			(at 153.67 93.98 0)
 			(effects
 				(font
@@
 		)
 		(property "Sim.Library" "${KICAD9_SYMBOL_DIR}/Simulation_SPICE.sp"
-			(at 157.48 36.83 0)
+			(at 153.67 93.98 0)
 			(effects
 				(font
@@
 		)
 		(property "Sim.Name" "kicad_builtin_opamp_dual"
-			(at 157.48 36.83 0)
+			(at 153.67 93.98 0)
 			(effects
 				(font
@@
 		)
 		(property "Sim.Device" "SUBCKT"
-			(at 157.48 36.83 0)
+			(at 153.67 93.98 0)
 			(effects
 				(font
@@
 		)
 		(property "Sim.Pins" "1=out1 2=in1- 3=in1+ 4=vee 5=in2+ 6=in2- 7=out2 8=vcc"
-			(at 157.48 36.83 0)
+			(at 153.67 93.98 0)
 			(effects
 				(font
@@
 	(symbol
 		(lib_id "Device:Opamp_Dual")
-		(at 156.21 57.15 0)
+		(at 157.48 36.83 0)
 		(unit 2)
 		(exclude_from_sim no)
@@
 		(fields_autoplaced yes)
 		(property "Reference" "U4"
-			(at 156.21 46.99 0)
+			(at 157.48 26.67 0)
 			(effects
 				(font
@@
 		)
 		(property "Value" "Opamp_Dual"
-			(at 156.21 49.53 0)
+			(at 157.48 29.21 0)
 			(effects
 				(font
@@
 		)
 		(property "Footprint" "PowerManagementBoard:SOIC127P600X175-8N"
-			(at 156.21 57.15 0)
+			(at 157.48 36.83 0)
 			(effects
 				(font
@@
 		)
 		(property "Datasheet" "https://4donline.ihs.com/images/VipMasterIC/IC/DIOD/DIOD-S-A0005046231/DIOD-S-A0005046231-1.pdf?hkey=6D3A4C79FDBF58556ACFDE234799DDF0"
-			(at 156.21 57.15 0)
+			(at 157.48 36.83 0)
 			(effects
 				(font
@@
 		)
 		(property "Description" "Dual operational amplifier"
-			(at 156.21 57.15 0)
+			(at 157.48 36.83 0)
 			(effects
 				(font
@@
 		)
 		(property "Sim.Library" "${KICAD9_SYMBOL_DIR}/Simulation_SPICE.sp"
-			(at 156.21 57.15 0)
+			(at 157.48 36.83 0)
 			(effects
 				(font
@@
 		)
 		(property "Sim.Name" "kicad_builtin_opamp_dual"
-			(at 156.21 57.15 0)
+			(at 157.48 36.83 0)
 			(effects
 				(font
@@
 		)
 		(property "Sim.Device" "SUBCKT"
-			(at 156.21 57.15 0)
+			(at 157.48 36.83 0)
 			(effects
 				(font
@@
 		)
 		(property "Sim.Pins" "1=out1 2=in1- 3=in1+ 4=vee 5=in2+ 6=in2- 7=out2 8=vcc"
-			(at 156.21 57.15 0)
+			(at 157.48 36.83 0)
 			(effects
 				(font
