File: BreakoutBoard/BattBreakout/BattBreakout.kicad_sch (KiCad schematic)
At the start: 22 parts, among them Q4 IPB180N10S4-02, Q9 IPB180N10S4-02, U2 LM5050MK-1_NOPB, U3 LM5050MK-1_NOPB

Commit message: Updated mosfet in schematic
Parts:
- added D1, D6: GRN, LED_SMD:LED_0201_0603Metric_Pad0.64x0.40mm_HandSolder, symbol Device:LED
- added Q1, Q2: BSS138, Package_TO_SOT_SMD:SOT-23W_Handsoldering, symbol Transistor_FET:BSS138
- added R1, R3: 6.8k, Resistor_SMD:R_0201_0603Metric_Pad0.64x0.40mm_HandSolder, symbol Device:R_US
Connections:
- net +24V: now also Q1.2 (S), Q2.2 (S)
- net GND: now also D1.1 (K), D6.1 (K)
- net at Q9.1 (G), U3.5 (GATE): now also Q2.1 (G)
- net at Q4.1 (G), U2.5 (GATE): now also Q1.1 (G)
- new net: D1.2 (A), R1.1
- new net: Q1.3 (D), R1.2
- new net: D6.2 (A), R3.1
- new net: Q2.3 (D), R3.2

Commit message: Fixed resistor footprints
Parts:
- R2, R39: footprint Resistor_SMD:R_0603_1608Metric_Pad0.98x0.95mm_HandSolder -> Resistor_SMD:R_0201_0603Metric_Pad0.64x0.40mm_HandSolder
Changed lines of the file:
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@@
 			)
 		)
-		(property "Footprint" "Resistor_SMD:R_0603_1608Metric_Pad0.98x0.95mm_HandSolder"
+		(property "Footprint" "Resistor_SMD:R_0201_0603Metric_Pad0.64x0.40mm_HandSolder"
 			(at 110.744 55.626 90)
 			(effects
@@
 			)
 		)
-		(property "Footprint" "Resistor_SMD:R_0603_1608Metric_Pad0.98x0.95mm_HandSolder"
+		(property "Footprint" "Resistor_SMD:R_0201_0603Metric_Pad0.64x0.40mm_HandSolder"
 			(at 113.284 126.746 90)
 			(effects
